File: hardware/kai_monitoring/kai_monitoring.kicad_pcb (KiCad board)
At the start: 2 copper layers, 75 x 106.5 mm, 21 parts, among them J1 LCD Display Socket, J10 SPI Additional, J11 Unused Socket, J12 3.3V DC Socket, J13 FPC 14 Pin 1 mm, J14 LCD 2.54 mm Pin, J15 Micro_SD_Card_Det1, J16 I2C Additional 3, J2 RS485 Socket, J3 5V DC Socket, J4 TTL UART Socket, J5 SHT45 Socket, J6 W5500 Left Socket, J7 W5500 Right Socket, J8 I2C Additional 1, J9 I2C Additional 2, U1 YD-ESP32-S3

Commit message: Updated the pcb
Parts:
- added C1: 100nf, Capacitor_SMD:C_0805_2012Metric, F.Cu at (81.5, 50.5)
- added G1: LOGO, LOGO, F.Cu at (69.0, 58.0)
- added J13: FPC 14 Pin 1 mm, Connector_FFC-FPC:Molex_200528-0140_1x14-1MP_P1.00mm_Horizontal, F.Cu at (58.0, 92.8)
- added J14: LCD 2.54 mm Pin, Connector_PinSocket_2.54mm:PinSocket_1x14_P2.54mm_Vertical, F.Cu at (50.3, 76.2)
- added R1: 10k, Resistor_SMD:R_0805_2012Metric, F.Cu at (83.5, 54.1)
- added R2: 10k, Resistor_SMD:R_0805_2012Metric, F.Cu at (86.5, 54.1)
- added R3: 10k, Resistor_SMD:R_0805_2012Metric, F.Cu at (89.5, 54.1)
- added R4: 10k, Resistor_SMD:R_0805_2012Metric, F.Cu at (92.5, 54.1)
- added REF**: BreakLine_9h_D0.5mm_P0.85mm, Panelization:BreakLine_9h_D0.5mm_P0.85mm, F.Cu at (63.5, 61.6)
- added REF**: BreakLine_9h_D0.5mm_P0.85mm, Panelization:BreakLine_9h_D0.5mm_P0.85mm, F.Cu at (63.5, 46.3)
- added REF**: BreakLine_9h_D0.5mm_P0.85mm, Panelization:BreakLine_9h_D0.5mm_P0.85mm, F.Cu at (63.5, 107.5)
- added REF**: BreakLine_9h_D0.5mm_P0.85mm, Panelization:BreakLine_9h_D0.5mm_P0.85mm, F.Cu at (63.5, 92.2)
- added REF**: BreakLine_9h_D0.5mm_P0.85mm, Panelization:BreakLine_9h_D0.5mm_P0.85mm, F.Cu at (63.5, 38.6)
- added REF**: BreakLine_9h_D0.5mm_P0.85mm, Panelization:BreakLine_9h_D0.5mm_P0.85mm, F.Cu at (63.5, 69.2)
- added REF**: BreakLine_9h_D0.5mm_P0.85mm, Panelization:BreakLine_9h_D0.5mm_P0.85mm, F.Cu at (63.5, 84.5)
- added REF**: BreakLine_9h_D0.5mm_P0.85mm, Panelization:BreakLine_9h_D0.5mm_P0.85mm, F.Cu at (63.5, 99.8)
- added REF**: BreakLine_1h_D0.5mm_P0.85mm, Panelization:BreakLine_1h_D0.5mm_P0.85mm, F.Cu at (63.5, 111.7)
- added REF**: BreakLine_9h_D0.5mm_P0.85mm, Panelization:BreakLine_9h_D0.5mm_P0.85mm, F.Cu at (59.3, 73.5)
- added REF**: BreakLine_9h_D0.5mm_P0.85mm, Panelization:BreakLine_9h_D0.5mm_P0.85mm, F.Cu at (63.5, 54.0)
- added REF**: BreakLine_9h_D0.5mm_P0.85mm, Panelization:BreakLine_9h_D0.5mm_P0.85mm, F.Cu at (51.6, 73.5)
- added REF**: BreakLine_9h_D0.5mm_P0.85mm, Panelization:BreakLine_9h_D0.5mm_P0.85mm, F.Cu at (63.5, 76.9)
- moved J14 135.5 mm to (50.3, 38.0)
- moved J13 110.6 mm to (58.0, 54.5), turned to 90 degrees
- moved J10 93.2 mm to (136.3, 82.3)
- moved J12 23.8 mm to (134.0, 59.8)
- moved J6 21.7 mm to (122.0, 125.8)
- moved J7 21.7 mm to (102.0, 125.8)
- moved J8 21.7 mm to (66.8, 92.3)
- moved J9 21.7 mm to (66.8, 105.8)
- moved H4 21.7 mm to (68.8, 34.3)
- moved J15 21.7 mm to (87.0, 39.9)
- moved J3 21.7 mm to (134.0, 47.8)
- moved H2 21.7 mm to (68.8, 130.8)
- moved J16 21.7 mm to (66.8, 119.4)
- moved J2 21.7 mm to (80.3, 132.3)
- moved J5 21.7 mm to (66.8, 78.8)
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Connections:
- U1 pad 10: /CS TOUCH -> /SPI3 SCK
- U1 pad 11: /LED LCD -> /SPI3 MOSI
- U1 pad 12: /DC/RS LCD -> /RST W5500
- U1 pad 13: /RST LCD -> /SPI3 MISO
- U1 pad 15: /SPI2 MOSI -> /IRQ TOUCH
- U1 pad 16: /SPI2 SCK -> /CS TOUCH
- U1 pad 17: /SPI2 MISO -> /LED LCD
- U1 pad 18: /I2C SDA -> /DC/RS LCD
- U1 pad 19: /I2C SCL -> /RST LCD
- U1 pad 20: /SPI3 MISO -> /CS LCD
- U1 pad 27: /RXD TTL -> /CD SD
- U1 pad 28: /TXD TTL -> /CS SD
- U1 pad 30: /CS LCD -> /CS Additional
- U1 pad 35: /CS SD -> /SPI2 MISO
- U1 pad 36: /CD SD -> /SPI2 SCK
- U1 pad 37: /CS Additional -> /SPI2 MOSI
- U1 pad 38: /UNUSED 3 -> /I2C SDA
- U1 pad 39: /UNUSED 2 -> /I2C SCL
- U1 pad 4: /SPI3 SCK -> /UNUSED 3
- U1 pad 40: /UNUSED 1 -> /RXD TTL
- U1 pad 41: /UNUSED 0 -> /TXD TTL
- U1 pad 5: /SPI3 MOSI -> /UNUSED 2
- U1 pad 6: /RST W5500 -> /UNUSED 1
- U1 pad 7: /INT W5500 -> /UNUSED 0
- U1 pad 9: /IRQ TOUCH -> /INT W5500
Routing:
- net /CS Additional: track 0.00 -> 133.8 mm, vias 0 -> 1
- net /SPI3 MISO: track 0.00 -> 117.1 mm
- net /SPI3 MOSI: track 0.00 -> 114.8 mm, vias 0 -> 1
- net /SPI3 SCK: track 0.00 -> 108.7 mm
- net /SPI2 MOSI: track 0.00 -> 90.8 mm, vias 0 -> 4
- net /SPI2 SCK: track 0.00 -> 85.5 mm, vias 0 -> 4
- net /I2C SCL: track 0.00 -> 82.9 mm
- net /RST W5500: track 0.00 -> 79.3 mm
- net /I2C SDA: track 0.00 -> 78.7 mm
- net /SPI2 MISO: track 0.00 -> 72.4 mm, vias 0 -> 4
- net /RST LCD: track 0.00 -> 69.7 mm
- net /DC/RS LCD: track 0.00 -> 66.2 mm
- net +3.3V: track 238.7 -> 303.2 mm, vias 0 -> 3
- net /LED LCD: track 0.00 -> 61.1 mm
- net /CS TOUCH: track 0.00 -> 55.8 mm
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- added copper zone on B.Cu, net GND
- added copper zone on F.Cu, net GND
Other:
- board size 75 x 106.5 mm -> 91 x 106.5 mm
- board text added: "Monitoring Module-0"

Commit message: Updated the pcb again
Parts:
- removed G1: LOGO, LOGO
- removed J10: SPI Additional, Connector_PinSocket_2.54mm:PinSocket_1x06_P2.54mm_Vertical
- removed the J13 at (58.0, 54.5)
- removed the J13 at (58.0, 92.8)
- removed the J14 at (50.3, 38.0)
- removed the J14 at (50.3, 76.2)
- removed REF** (x12): BreakLine_9h_D0.5mm_P0.85mm, Panelization:BreakLine_9h_D0.5mm_P0.85mm
- removed REF**: BreakLine_1h_D0.5mm_P0.85mm, Panelization:BreakLine_1h_D0.5mm_P0.85mm
- added J13: FPC 14 Pin 1 mm, Connector_FFC-FPC:Molex_200528-0140_1x14-1MP_P1.00mm_Horizontal, F.Cu at (56.8, 65.4)
- added J14: LCD 2.54 mm Pin, Connector_PinSocket_2.54mm:PinSocket_1x14_P2.54mm_Vertical, F.Cu at (50.9, 48.8)
- added J17: LCD 2.54 mm Pin, Connector_PinSocket_2.54mm:PinSocket_1x14_P2.54mm_Vertical, F.Cu at (51.0, 90.5)
- added J18: FPC 14 Pin 1 mm, Connector_FFC-FPC:Molex_200528-0140_1x14-1MP_P1.00mm_Horizontal, F.Cu at (57.1, 107.0)
- moved R4 2.00 mm to (94.5, 54.1)
- moved R3 1.50 mm to (91.0, 54.1)
- moved J12 1.00 mm to (133.0, 59.6)
- moved C1 1.00 mm to (82.5, 50.5)
- moved R2 1.00 mm to (87.5, 54.1)
- moved J3 0.97 mm to (133.0, 47.8)
- moved R1 0.50 mm to (84.0, 54.1)
Routing:
- net GND: track 355.6 -> 6.75 mm
- net /CS Additional: track 133.8 -> 0.00 mm, vias 1 -> 0
- net /SPI3 SCK: track 108.7 -> 61.8 mm
- net /SPI3 MOSI: track 114.8 -> 68.0 mm, vias 1 -> 0
- net /SPI3 MISO: track 117.1 -> 76.5 mm
- net Net-(J13-Pin_14): track 32.7 -> 13.9 mm
- net Net-(J13-Pin_1): track 32.4 -> 13.8 mm
- net Net-(J13-Pin_13): track 29.1 -> 12.3 mm
- net Net-(J13-Pin_2): track 29.2 -> 12.7 mm
- net Net-(J13-Pin_12): track 26.8 -> 11.4 mm
- net Net-(J13-Pin_3): track 26.3 -> 10.9 mm
- net Net-(J17-Pin_1): track 0.00 -> 13.9 mm
- net Net-(J17-Pin_14): track 0.00 -> 13.8 mm
- net Net-(J13-Pin_4): track 22.7 -> 9.12 mm
- net Net-(J13-Pin_11): track 22.9 -> 9.48 mm
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Other:
- board size 91 x 106.5 mm -> 89.9 x 106.5 mm
- board text added: "Monitoring Module v1.0"
- board text removed: "CS (40)"
- board text removed: "Monitoring Module-0"
