File: hardware/kai_monitoring/kai_monitoring.kicad_sch (KiCad schematic)
At the start: 21 parts, among them J1 LCD Display Socket, J10 SPI Additional, J11 Unused Socket, J12 3.3V DC Socket, J13 FPC 14 Pin 1 mm, J14 LCD 2.54 mm Pin, J15 Micro_SD_Card_Det1, J16 I2C Additional 3, J2 RS485 Socket, J3 5V DC Socket, J4 TTL UART Socket, J5 SHT45 Socket, J6 W5500 Left Socket, J7 W5500 Right Socket, J8 I2C Additional 1, J9 I2C Additional 2, U1 YD-ESP32-S3

Commit message: Updated the pcb
Parts:
- added C1: 100nf, Capacitor_SMD:C_0805_2012Metric, symbol Device:C
- added R1, R2, R3, R4: 10k, Resistor_SMD:R_0805_2012Metric, symbol Device:R
Connections:
- net +3.3V: now also C1.1, R1.1, R2.1, R3.1, R4.1
- net CD SD: now also U1.27 (GPIO21); no longer U1.36 (GPIO39)
- net CS Additional: now also U1.30 (GPIO45); no longer U1.37 (GPIO40)
- net CS LCD: now also U1.20 (GPIO14); no longer U1.30 (GPIO45)
- net CS SD: now also U1.28 (GPIO47), R1.2; no longer U1.35 (GPIO38)
- net CS TOUCH: now also U1.16 (GPIO10); no longer U1.10 (GPIO17)
- net DC/RS LCD: now also U1.18 (GPIO12); no longer U1.12 (GPIO8)
- net GND: now also C1.2
- net I2C SCL: now also U1.39 (GPIO42); no longer U1.19 (GPIO13)
- net I2C SDA: now also U1.38 (GPIO41); no longer U1.18 (GPIO12)
- net INT W5500: now also U1.9 (GPIO16); no longer U1.7 (GPIO7)
- net IRQ TOUCH: now also U1.15 (GPIO9); no longer U1.9 (GPIO16)
- net LED LCD: now also U1.17 (GPIO11); no longer U1.11 (GPIO18)
- net RST LCD: now also U1.19 (GPIO13); no longer U1.13 (GPIO3)
- net RST W5500: now also U1.12 (GPIO8); no longer U1.6 (GPIO6)
- net RXD TTL: now also U1.40 (GPIO2); no longer U1.27 (GPIO21)
- net SPI2 MISO: now also U1.35 (GPIO38), R4.2; no longer U1.17 (GPIO11)
- net SPI2 MOSI: now also U1.37 (GPIO40), R2.2; no longer U1.15 (GPIO9)
- net SPI2 SCK: now also U1.36 (GPIO39), R3.2; no longer U1.16 (GPIO10)
- net SPI3 MISO: now also U1.13 (GPIO3); no longer U1.20 (GPIO14)
- net SPI3 MOSI: now also U1.11 (GPIO18); no longer U1.5 (GPIO5)
- net SPI3 SCK: now also U1.10 (GPIO17); no longer U1.4 (GPIO4)
- net TXD TTL: now also U1.41 (GPIO1); no longer U1.28 (GPIO47)
- net UNUSED 0: now also U1.7 (GPIO7); no longer U1.41 (GPIO1)
- net UNUSED 1: now also U1.6 (GPIO6); no longer U1.40 (GPIO2)
- net UNUSED 2: now also U1.5 (GPIO5); no longer U1.39 (GPIO42)
- net UNUSED 3: now also U1.4 (GPIO4); no longer U1.38 (GPIO41)

Commit message: Updated the pcb again
Parts:
- removed H1, H2, H3, H4: MountingHole, MountingHole:MountingHole_3.2mm_M3_Pad, symbol Mechanical:MountingHole
- removed J10: SPI Additional, Connector_PinSocket_2.54mm:PinSocket_1x06_P2.54mm_Vertical, symbol Connector:Conn_01x06_Socket
- added H1, H2, H3, H4: MountingHole_Pad, symbol Mechanical:MountingHole_Pad
- added J17: LCD 2.54 mm Pin, Connector_PinSocket_2.54mm:PinSocket_1x14_P2.54mm_Vertical, symbol Connector:Conn_01x14_Socket
- added J18: FPC 14 Pin 1 mm, Connector_FFC-FPC:Molex_200528-0140_1x14-1MP_P1.00mm_Horizontal, symbol Connector:Conn_01x14_Socket
Connections:
- net GND: now also H1.1, H2.1, H3.1, H4.1
- new net: J17.14 (Pin_14), J18.1 (Pin_1)
- new net: J17.5 (Pin_5), J18.10 (Pin_10)
- new net: J17.4 (Pin_4), J18.11 (Pin_11)
- new net: J17.3 (Pin_3), J18.12 (Pin_12)
- new net: J17.2 (Pin_2), J18.13 (Pin_13)
- new net: J17.1 (Pin_1), J18.14 (Pin_14)
- new net: J17.13 (Pin_13), J18.2 (Pin_2)
- new net: J17.12 (Pin_12), J18.3 (Pin_3)
- new net: J17.11 (Pin_11), J18.4 (Pin_4)
- new net: J17.10 (Pin_10), J18.5 (Pin_5)
- new net: J17.9 (Pin_9), J18.6 (Pin_6)
- new net: J17.8 (Pin_8), J18.7 (Pin_7)
- new net: J17.7 (Pin_7), J18.8 (Pin_8)
- new net: J17.6 (Pin_6), J18.9 (Pin_9)
